Commit message: 3 tane imu sensörü tanımlandı ve gazeboda simule edildi

File: imu_example/urdf/my_robot.urdf.xacro (robot description, xacro)
@@ -4,56 +4,49 @@
     <xacro:include filename="$(find imu_example)/urdf/robot_materials.xacro" />
     <xacro:include filename="$(find imu_example)/urdf/robot_gazebo.xacro" />
+    <xacro:include filename="$(find imu_example)/urdf/robot_gazebo_controls.xacro"/>
     <link name="base_footprint" />
-    <xacro:base_link />
+    <xacro:vehicle_body />
     <joint name="base_joint" type="fixed">
         <parent link="base_footprint"/>
-        <child link="base_link"/>
-        <origin xyz="0 0 0.1"/>
+        <child link="vehicle_body"/>
+        <origin xyz="0 0 ${body_height / 2}"/>
     </joint>
-    <xacro:wheel prefix="front_right" />
-    <xacro:wheel prefix="front_left" />
     <xacro:wheel prefix="rear_right" />
     <xacro:wheel prefix="rear_left" />
-    <joint name="front_right_wheel_joint" type="continuous">
-        <parent link="base_link"/>
-        <child link="front_right_wheel"/>
-        <origin xyz="0.2 0.275 0" rpy="${pi/2} 0 0"/>
-        <axis xyz="1 0 0"/>
-    </joint>
-    <joint name="front_left_wheel_joint" type="continuous">
-        <parent link="base_link"/>
-        <child link="front_left_wheel"/>
-        <origin xyz="0.2 -0.275 0" rpy="${pi/2} 0 0"/>
-        <axis xyz="1 0 0"/>
-    </joint>
+    <xacro:caster_wheel prefix="front" />
     <joint name="rear_right_wheel_joint" type="continuous">
-        <parent link="base_link"/>
+        <parent link="vehicle_body"/>
         <child link="rear_right_wheel"/>
-        <origin xyz="-0.2 0.275 0" rpy="${pi/2} 0 0"/>
-        <axis xyz="1 0 0"/>
+        <origin xyz="${-(body_width / 4)} ${((body_depth / 2) + (wheel_length / 2))} 0" rpy="${pi/2} 0 0"/>
+        <axis xyz="0 0 1"/>
     </joint>
     <joint name="rear_left_wheel_joint" type="continuous">
-        <parent link="base_link"/>
+        <parent link="vehicle_body"/>
         <child link="rear_left_wheel"/>
-        <origin xyz="-0.2 -0.275 0" rpy="${pi/2} 0 0"/>
-        <axis xyz="1 0 0"/>
+        <origin xyz="${-(body_width / 4)} ${-((body_depth / 2) + (wheel_length / 2))} 0" rpy="${pi/2} 0 0"/>
+        <axis xyz="0 0 1"/>
     </joint>
-    <xacro:imu prefix="1" />
-    <xacro:imu prefix="2" />
-    <xacro:imu prefix="3" />
+    <joint name="front_caster_wheel_joint" type="fixed">
+        <parent link="vehicle_body"/>
+        <child  link="front_caster_wheel"/>
+        <origin xyz="${body_width / 4} 0 0"/>
+    </joint>
+    <xacro:imu prefix="imu1" />
+    <xacro:imu prefix="imu2" />
+    <xacro:imu prefix="imu3" />
     <joint name="imu_joint_1" type="fixed">
-        <parent link="base_link"/>
-        <child link="1_imu"/>
-        <origin xyz="0 0 0.05"/>
+        <parent link="vehicle_body"/>
+        <child link="imu1_link"/>
+        <origin xyz="${body_width / 4} 0 ${(body_height / 2) + 0.01 + wheel_radius}" rpy="0 0 0"/>
     </joint>
     <joint name="imu_joint_2" type="fixed">
-        <parent link="base_link"/>
-        <child link="2_imu"/>
-        <origin xyz="0.2 0 0.05"/>
+        <parent link="vehicle_body"/>
+        <child link="imu2_link"/>
+        <origin xyz="0 0 ${(body_height / 2) + 0.01 + wheel_radius}"/>
     </joint>
     <joint name="imu_joint_3" type="fixed">
-        <parent link="base_link"/>
-        <child link="3_imu"/>
-        <origin xyz="-0.2 0 0.05"/>
+        <parent link="vehicle_body"/>
+        <child link="imu3_link"/>
+        <origin xyz="${-(body_width / 4)} 0 ${(body_height / 2) + 0.01 + wheel_radius}"/>
     </joint>
 </robot>

File: imu_example/urdf/robot_gazebo.xacro (robot description, xacro)
@@ -1,5 +1,35 @@
 <?xml version="1.0"?>
-<robot name="my_robot" xmlns="http://ros.org/wiki/xacro">
+<robot name="my_robot" xmlns="http://www.ros.org/wiki/xacro">
+    <gazebo references="$rear_right_wheel">
+        <mu1>10000</mu1>
+        <mu2>10000</mu2>
+        <kp>10000</kp>
+        <kd>10.0</kd>
+        <minDepth>0.001</minDepth>
+        <maxVel>0.1</maxVel>
+        <fdirl>1 0 0</fdirl>
+    </gazebo>
+    <gazebo references="$rear_left_wheel">
+        <mu1>10000</mu1>
+        <mu2>10000</mu2>
+        <kp>10000</kp>
+        <kd>10.0</kd>
+        <minDepth>0.001</minDepth>
+        <maxVel>0.1</maxVel>
+        <fdirl>1 0 0</fdirl>
+    </gazebo>
+    <gazebo references="front_caster_wheel">
+        <mu1>0.1</mu1>
+        <mu2>0.1</mu2>
+        <kp>1000000.0</kp>
+        <kd>100.0</kd>
+        <minDepth>0.001</minDepth>
+        <maxVel>0.1</maxVel>
+        <fdirl>1 0 0</fdirl>
+    </gazebo>
     <gazebo>
+        <plugin filename="ign_ros2_control-system" name="ign_ros2_control::IgnitionROS2ControlPlugin">
+            <parameters>$(find imu_example)/config/robot_controller.yaml</parameters>
+        </plugin>
         <plugin filename="ignition-gazebo-imu-system" name="ignition::gazebo::systems::Imu"/>
         <plugin filename="ignition-gazebo-sensors-system" name="ignition::gazebo::systems::Sensors">

File: imu_example/urdf/robot_materials.xacro (robot description, xacro)
@@ -4,4 +4,12 @@
     <xacro:property name="wheel_radius" value="0.1"/>
     <xacro:property name="wheel_length" value="0.05" />
+    <xacro:property name="wheel_mass" value="0.5" />
+    <xacro:property name="caster_wheel_radius" value="0.1" />
+    <xacro:property name="caster_wheel_mass" value="0.5"/>
+    <!-- Vehicle Body Parameters -->
+    <xacro:property name="body_width"  value="0.6" />
+    <xacro:property name="body_depth"  value="0.5" />
+    <xacro:property name="body_height" value="0.2" />
+    <xacro:property name="body_mass" value="2" />
     <xacro:macro name="wheel" params="prefix">
         <link name="${prefix}_wheel">
@@ -21,5 +29,5 @@
             <inertial>
                 <origin xyz="0 0 0" rpy="0 0 0"/>
-                <mass value="1" />
+                <mass value="${wheel_mass}" />
                 <inertia ixx="${(1 / 12) * ((3 * wheel_radius * wheel_radius) + (wheel_length * wheel_length))}"
                          iyy="${(1 / 12) * ((3 * wheel_radius * wheel_radius) + (wheel_length * wheel_length))}"
@@ -29,35 +37,52 @@
             </inertial>
         </link>
-        <gazebo references="${prefix}_wheel">
-            <mu1>10000</mu1>
-            <mu2>10000</mu2>
-            <kp>10000</kp>
-            <kd>10.0</kd>
-            <minDepth>0.001</minDepth>
-            <maxVel>0.1</maxVel>
-            <fdirl>1 0 0</fdirl>
-        </gazebo>
     </xacro:macro>
-    <xacro:macro name="base_link">
-        <link name="base_link">
+    <xacro:macro name="caster_wheel" params="prefix">
+        <link name="${prefix}_caster_wheel">
             <visual>
-                <origin xyz ="0 0 0" />
+                <origin xyz="0 0 0"/>
                 <geometry>
-                    <box size="0.8 0.5 0.1"/>
+                    <sphere radius="${caster_wheel_radius}"/>
+                </geometry>
+                <material name="black"/>
+            </visual>
+            <collision>
+                <origin xyz="0 0 0"/>
+                <geometry>
+                    <sphere radius="${caster_wheel_radius}"/>
+                </geometry>
+            </collision>
+            <inertial>
+                <origin xyz="0 0 0"/>
+                <mass value="${caster_wheel_mass}" />
+                <inertia ixx="${(2 / 5) * (caster_wheel_mass * caster_wheel_radius * caster_wheel_radius)}"
+                         iyy="${(2 / 5) * (caster_wheel_mass * caster_wheel_radius * caster_wheel_radius)}"
+                         izz="${(2 / 5) * (caster_wheel_mass * caster_wheel_radius * caster_wheel_radius)}"
+                         ixy = "0" ixz="0" iyz="0" iyx="0" izx="0" izy="0"
+                />
+            </inertial>
+        </link>
+    </xacro:macro>
+    <xacro:macro name="vehicle_body">
+        <link name="vehicle_body">
+            <visual>
+                <origin xyz ="0 0 ${wheel_radius}" />
+                <geometry>
+                    <box size="${body_width} ${body_depth} ${body_height}"/>
                 </geometry>
                 <material name="red"/>
             </visual>
             <collision>
-                <origin xyz ="0 0 0" />
+                <origin xyz ="0 0 ${wheel_radius}" />
                 <geometry>
-                    <box size="0.8 0.5 0.1"/>
+                     <box size="${body_width} ${body_depth} ${body_height}"/>
                 </geometry>
             </collision>
             <inertial>
                 <origin xyz="0 0 0" rpy="0 0 0"/>
-                <mass value="7"/>
-                <inertia ixx="${(1 / 12) * 7 * (0.5 * 0.5 + 0.1 * 0.1)}"
-                        iyy="${(1 / 12) * 7 * (0.8 * 0.8 + 0.1 * 0.1)}"
-                        izz="${(1 / 12) * 7 * (0.8 * 0.8 + 0.5 * 0.5)}"
+                <mass value="${body_mass}"/>
+                <inertia ixx="${(1 / 12) * body_mass * (body_height * body_height + body_depth * body_depth)}"
+                        iyy="${(1 / 12) * body_mass * (body_height * body_height + body_width * body_width)}"
+                        izz="${(1 / 12) * body_mass * (body_width * body_width + body_depth * body_depth)}"
                         ixy = "0" ixz="0" iyz="0" iyx="0" izx="0" izy="0"
                 />
@@ -66,5 +91,5 @@
     </xacro:macro>
     <xacro:macro name="imu" params="prefix">
-        <link name="${prefix}_imu">
+        <link name="${prefix}_link">
             <visual>
                 <origin xyz="0 0 0"/>
@@ -82,5 +107,5 @@
             <inertial>
                 <origin xyz="0 0 0" rpy="0 0 0" />
-                <mass value="0.4" />
+                <mass value="0.1" />
                 <inertia ixx="${(1 / 12) * 0.4 * (0.05 * 0.05 + 0.02 * 0.02)}"
                          iyy="${(1 / 12) * 0.4 * (0.05 * 0.05 + 0.02 * 0.02)}"
@@ -90,19 +115,10 @@
             </inertial>
         </link>
-        <gazebo references="${prefix}_imu">
-            <sensor name="imu" type="imu">
+        <gazebo reference="${prefix}_link">
+            <sensor name="${prefix}" type="imu">
                 <always_on>true</always_on>
                 <update_rate>100</update_rate>
-                <gz_frame_id>${prefix}_imu</gz_frame_id>
-                <topic>${prefix}_imu</topic>
-                <imu>
-                    <noise>
-                        <type>gaussian</type>
-                        <mean>0.0</mean>
-                        <stddev>0.01</stddev>
-                    </noise>
-                    <orientation_reference_frame>world</orientation_reference_frame>
-                    <gravity>true</gravity>
-                </imu>
+                <gz_frame_id>${prefix}_link</gz_frame_id>
+                <topic>${prefix}</topic>
             </sensor>
         </gazebo>

Commit message: Imu verileri düzgünce okunuyor ve yeni bir dünya tanımlandı

File: imu_example/urdf/my_robot.urdf.xacro (robot description, xacro)
@@ -18,5 +18,5 @@
         <parent link="vehicle_body"/>
         <child link="rear_right_wheel"/>
-        <origin xyz="${-(body_width / 4)} ${((body_depth / 2) + (wheel_length / 2))} 0" rpy="${pi/2} 0 0"/>
+        <origin xyz="${-(body_width / 4)} ${((body_depth / 2) + (wheel_length / 2))} 0" rpy="-${pi/2} 0 0"/>
         <axis xyz="0 0 1"/>
     </joint>
@@ -24,5 +24,5 @@
         <parent link="vehicle_body"/>
         <child link="rear_left_wheel"/>
-        <origin xyz="${-(body_width / 4)} ${-((body_depth / 2) + (wheel_length / 2))} 0" rpy="${pi/2} 0 0"/>
+        <origin xyz="${-(body_width / 4)} ${-((body_depth / 2) + (wheel_length / 2))} 0" rpy="-${pi/2} 0 0"/>
         <axis xyz="0 0 1"/>
     </joint>

Commit message: Imu verileri dosyaya loglandı!

File: imu_example/urdf/my_robot.urdf.xacro (robot description, xacro)
@@ -38,5 +38,5 @@
         <parent link="vehicle_body"/>
         <child link="imu1_link"/>
-        <origin xyz="${body_width / 4} 0 ${(body_height / 2) + 0.01 + wheel_radius}" rpy="0 0 0"/>
+        <origin xyz="${0.05} 0 ${(body_height / 2) + 0.01 + wheel_radius}" rpy="0 0 0"/>
     </joint>
     <joint name="imu_joint_2" type="fixed">
@@ -48,5 +48,5 @@
         <parent link="vehicle_body"/>
         <child link="imu3_link"/>
-        <origin xyz="${-(body_width / 4)} 0 ${(body_height / 2) + 0.01 + wheel_radius}"/>
+        <origin xyz="${-0.05} 0 ${(body_height / 2) + 0.01 + wheel_radius}"/>
     </joint>
 </robot>
